File: circuit_board/SensorDemo/SensorDemo.kicad_pcb (KiCad board)
At the start: 4 copper layers, 46 x 68 mm, 72 parts, among them K1 PB_SMD, P1 TC2050_IDC_NL, U1 TLV1117-33CDCYR, U2 dsPIC33EP32GP502, U3 LTC1658, U4 INA333, U5 REF1925, U6 REF1925, X1 8MHz

Commit message: updated fiducial marks
Parts:
- removed the FD at (123.0, 62.5)
- added FD: Val**, SensorDemo_pcb:FD_1MM_CR, F.Cu at (123.0, 62.5)
- FD (x2): footprint SensorDemo_pcb:FD_1MM_R -> SensorDemo_pcb:FD_1MM_CR
- FD (x3): footprint SensorDemo_pcb:FD_1MM_C -> SensorDemo_pcb:FD_1MM_SQ
